File: coil_tempeauture_interlock-backups/coil_tempeauture_interlock-2025-06-07_165229/coil_tempeauture_interlock.kicad_sch (KiCad schematic)
At the start: 41 parts, among them J1 Conn_01x10_Pin, J10 -12V, J11 +12V, J2 Conn_01x10_Pin, J4 Conn_01x05, J6 Output1, J7 Output2, J8 Thermalcouple1, J9 Thermocouple2, Q1 BS107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

Commit message: update interlock with AD620
Parts:
- J10: value -12V -> Conn_Coaxial
- J11: value +12V -> Conn_Coaxial
- J6: value Output1 -> Conn_Coaxial
- J7: value Output2 -> Conn_Coaxial
- J8: value Thermalcouple1 -> Conn_Coaxial
- J9: value Thermocouple2 -> Conn_Coaxial
- R1: value 470R -> 5R; LCSC C119317 -> C334308
- R2: value 5.1k -> 47k; LCSC C58591 -> C2857423
- RV1: value 20k -> 100k; LCSC C34845 -> C118963
Connections:
- net +12V: no longer J11.1 (In)
- net -12V: no longer J10.1 (In)
- net GND: no longer J10.2 (Ext), J11.2 (Ext)
- net Set: no longer R1.2, RV1.2, RV1.3
- new net Ref: R1.2, RV1.2, RV1.3
Other:
- moved on the sheet: J10, J11, J4
