File: coil_tempeauture_interlock.kicad_pcb (KiCad board)
At the start: 4 copper layers, 100 x 100 mm, 32 parts, among them J1 Conn_01x10_Pin, J10 Conn_Coaxial, J11 Conn_Coaxial, J12 Conn_01x04_Pin, J2 Conn_01x10_Pin, J3 Conn_01x04_Pin, J4 Conn_01x05, J5 Conn_01x03, J6 Conn_Coaxial, J7 Conn_Coaxial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

Commit message: update interlock with AD620
Parts:
- removed C2: 1u, Capacitor_THT:C_Disc_D4.3mm_W1.9mm_P5.00mm
- removed H1, H2: Keystone Electronics 621, matterwaves:Keystone 621
- removed J12, J3: Conn_01x04_Pin, Connector_JST:JST_PH_S4B-PH-K_1x04_P2.00mm_Horizontal
- removed J5: Conn_01x03, Connector_Wire:SolderWire-0.75sqmm_1x03_P4.8mm_D1.25mm_OD2.3mm
- removed R5: 100k, Resistor_THT:R_Axial_DIN0207_L6.3mm_D2.5mm_P10.16mm_Horizontal
- added C10: 100n, Capacitor_THT:C_Disc_D4.3mm_W1.9mm_P5.00mm, F.Cu at (172.7, 116.8)
- added C11: 100n, Capacitor_THT:C_Disc_D4.3mm_W1.9mm_P5.00mm, F.Cu at (154.9, 121.9)
- added C12: 10u, Capacitor_THT:C_Disc_D4.3mm_W1.9mm_P5.00mm, F.Cu at (152.4, 121.9)
- added C13: 1u, Capacitor_THT:C_Disc_D4.3mm_W1.9mm_P5.00mm, F.Cu at (162.0, 129.5)
- added C5: 10u, Capacitor_THT:C_Disc_D4.3mm_W1.9mm_P5.00mm, F.Cu at (152.4, 116.8)
- added C6: 100n, Capacitor_THT:C_Disc_D4.3mm_W1.9mm_P5.00mm, F.Cu at (154.9, 116.8)
- added C7: 10u, Capacitor_THT:C_Disc_D4.3mm_W1.9mm_P5.00mm, F.Cu at (132.1, 121.9)
- added C8: 100n, Capacitor_THT:C_Disc_D4.3mm_W1.9mm_P5.00mm, F.Cu at (134.6, 121.9)
- added C9: 10u, Capacitor_THT:C_Disc_D4.3mm_W1.9mm_P5.00mm, F.Cu at (175.3, 116.8)
- added R10: 100R, Resistor_THT:R_Axial_DIN0207_L6.3mm_D2.5mm_P10.16mm_Horizontal, F.Cu at (167.6, 109.2)
- added R11: 100R, Resistor_THT:R_Axial_DIN0207_L6.3mm_D2.5mm_P10.16mm_Horizontal, F.Cu at (167.6, 104.1)
- added R7: 100R, Resistor_THT:R_Axial_DIN0207_L6.3mm_D2.5mm_P10.16mm_Horizontal, F.Cu at (147.3, 104.1)
- added R8: 100R, Resistor_THT:R_Axial_DIN0207_L6.3mm_D2.5mm_P10.16mm_Horizontal, F.Cu at (147.3, 109.2)
- added R9: 100k, Resistor_THT:R_Axial_DIN0207_L6.3mm_D2.5mm_P10.16mm_Horizontal, F.Cu at (158.0, 139.7)
- added U2: AD620, Package_DIP:DIP-8_W7.62mm_Socket_LongPads, F.Cu at (139.7, 114.3)
- added U3: AD620, Package_DIP:DIP-8_W7.62mm_Socket_LongPads, F.Cu at (160.0, 114.3)
- J10: value Conn_Coaxial -> -12V
- J11: value Conn_Coaxial -> +12V
- J6: value Conn_Coaxial -> Output1
- J7: value Conn_Coaxial -> Output2
- J8: value Conn_Coaxial -> Thermalcouple1
- J9: value Conn_Coaxial -> Thermocouple2
- R1: value 5R -> 470R
- R2: value 47k -> 5.1k
- RV1: value 100k -> 20k
- moved R3 40.9 mm to (142.0, 139.7), turned to 90 degrees
- moved C4 28.6 mm to (160.1, 88.9)
- moved C1 23.5 mm to (146.0, 129.5), turned to -90 degrees
- moved C3 22.8 mm to (160.1, 91.4)
- moved U1 22.7 mm to (147.3, 91.4)
- moved R6 12.4 mm to (124.5, 121.9)
- moved R1 9.97 mm to (129.5, 81.3)
- moved R2 9.76 mm to (165.1, 81.3)
- moved RV1 9.53 mm to (149.9, 81.3)
- moved Q1 6.99 mm to (111.8, 127.0)
- moved R4 6.37 mm to (114.3, 121.9)
- moved Q2 5.29 mm to (124.5, 127.0)
Connections:
- net /Ref renamed /Set
- C1 pad 1: Net-(Q1-G) -> Net-(U2-+)
- J10 pad 1: unconnected-(J10-In-Pad1) -> -12V
- J10 pad 2: unconnected-(J10-Ext-Pad2) -> GND
- J11 pad 1: unconnected-(J11-In-Pad1) -> +12V
- J11 pad 2: unconnected-(J11-Ext-Pad2) -> GND
- R3 pad 1: Net-(U1A-OUT) -> Net-(J8-In)
- R3 pad 2: Net-(Q1-G) -> Net-(U2-+)
- U1 pad 1: Net-(U1A-OUT) -> Net-(Q1-G)
- U1 pad 2: Net-(J8-In) -> Net-(U1A--IN)
- U1 pad 6: Net-(J9-In) -> Net-(U1B--IN)
- U1 pad 7: Net-(U1B-OUT) -> Net-(Q2-G)
Routing:
- net GND: track 286.5 -> 105.6 mm
- net -12V: track 47.5 -> 195.2 mm
- net +12V: track 128.2 -> 234.6 mm
- net Net-(U1A-OUT): track 49.0 -> 0.00 mm
- net Net-(U1B-OUT): track 36.2 -> 0.00 mm
- net Net-(Q1-G): track 17.5 -> 51.3 mm
- net Net-(J8-In): track 39.5 -> 7.23 mm
- net Net-(Q2-G): track 17.9 -> 47.7 mm
- net /I2C_SCL: track 28.5 -> 0.00 mm
- net Net-(U1B--IN): track 0.00 -> 28.1 mm
- net Net-(U1A--IN): track 0.00 -> 27.5 mm
- net Net-(J9-In): track 33.5 -> 7.23 mm
- net /I2C_SDA: track 20.5 -> 0.00 mm
- net GNDS: track 19.1 -> 0.00 mm
- net VBUS: track 16.0 -> 0.00 mm
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- added copper zone on B.Cu, net GND
- added copper zone on F.Cu, net GND
- added copper zone on In1.Cu, net GND
- added copper zone on In2.Cu, net GND
Other:
- board text added: "2 Channel Temperature Interlock"
- board text added: "Mueller Group, UC Berkeley"
- board text removed: "CIRCUIT NAME"
- board text removed: "I^{2}C GND"
- board text removed: "J Roth, Mueller Group, UC Berkeley"
- board text removed: "SCL"
- board text removed: "SDA"
- board text removed: "STEMMA"

Commit message: isolate thermocouple input
Connections:
- J8 pad 2: GND -> Net-(J8-Ext)
- J9 pad 2: GND -> Net-(J9-Ext)
- U2 pad 2: GND -> Net-(J8-Ext)
- U3 pad 2: GND -> Net-(J9-Ext)
Routing:
- net Net-(J9-Ext): track 0.00 -> 28.9 mm
- net Net-(J8-Ext): track 0.00 -> 27.5 mm
